File: board/E4m.brd (EAGLE design)
At the start: 49.4 x 100.1 mm, 76 parts, among them IC1 MCP23017SS, Q1 IRL540, Q2 IRL540, Q3 IRL540

Commit message: 100% routed..... to clean before raster...
yup
Routing:
- net GND: track 0.23 -> 310.8 mm, vias 0 -> 3
- net 3V3: track 0.18 -> 186.3 mm, vias 0 -> 4
- net 12V: track 0.00 -> 171.6 mm
- net N$27: track 0.00 -> 114.4 mm, vias 0 -> 3
- net 5V: track 0.00 -> 103.8 mm, vias 0 -> 2
- net N$S4: track 0.00 -> 89.5 mm, vias 0 -> 2
- net ENABLE: track 0.00 -> 81.1 mm, vias 0 -> 1
- net N$23: track 0.00 -> 76.2 mm, vias 0 -> 4
- net GND1: track 0.00 -> 63.6 mm, vias 0 -> 1
- net E-STEP: track 0.00 -> 56.5 mm, vias 0 -> 3
- net ANALOG: track 0.00 -> 49.5 mm
- net X-DIR: track 0.00 -> 40.8 mm, vias 0 -> 1
- net E-DIR: track 0.00 -> 39.0 mm, vias 0 -> 3
- net 12V1: track 0.00 -> 35.2 mm, vias 0 -> 1
- net SCL: track 0.00 -> 34.4 mm, vias 0 -> 2
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- removed copper zone on layer 1, net GND
- removed copper zone on layer 16, net GND
- removed copper zone on layer 1, net GND1
- removed copper zone on layer 16, net GND1

Commit message: again
again
Routing:
- net 12V: track 171.6 -> 173.1 mm
Changed lines of the file:
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@@
 <wire x1="11.58875" y1="35.8775" x2="12.065" y2="35.8775" width="0.254" layer="1"/>
 <wire x1="12.065" y1="35.8775" x2="12.197" y2="35.756" width="0.254" layer="1"/>
-<wire x1="13.49375" y1="41.43375" x2="13.49375" y2="42.8625" width="0.254" layer="1"/>
-<wire x1="11.58875" y1="39.52875" x2="11.668125" y2="39.608125" width="0.254" layer="1"/>
-<wire x1="11.668125" y1="39.608125" x2="13.49375" y2="41.43375" width="0.254" layer="1"/>
+<wire x1="13.51915" y1="41.91635" x2="13.49375" y2="42.8625" width="0.254" layer="1"/>
+<wire x1="11.58875" y1="39.52875" x2="11.591925" y2="40.039925" width="0.254" layer="1"/>
+<wire x1="11.591925" y1="40.039925" x2="13.51915" y2="41.91635" width="0.254" layer="1"/>
 <wire x1="11.58875" y1="35.8775" x2="11.58875" y2="39.52875" width="0.254" layer="1"/>
 <wire x1="13.49375" y1="42.8625" x2="13.497" y2="43.006" width="0.254" layer="1"/>
@@
 <wire x1="4.60375" y1="44.1325" x2="4.7498" y2="44.0182" width="0.254" layer="1"/>
 <wire x1="2.2225" y1="44.1325" x2="2.2098" y2="44.0182" width="0.254" layer="1"/>
-<wire x1="7.3025" y1="43.97375" x2="11.668125" y2="39.608125" width="0.254" layer="1"/>
+<wire x1="7.3025" y1="43.97375" x2="11.591925" y2="40.039925" width="0.254" layer="1"/>
 <wire x1="7.3025" y1="43.97375" x2="7.2898" y2="44.0182" width="0.254" layer="1"/>
 <wire x1="6.6675" y1="80.01" x2="6.6675" y2="78.74" width="0.254" layer="1"/>
@@
 <contactref element="PAD2" pad="1"/>
 <wire x1="16.097" y1="43.006" x2="16.097" y2="40.1132" width="0.254" layer="1"/>
-<wire x1="16.097" y1="40.1132" x2="17.1704" y2="39.0144" width="0.254" layer="1"/>
-<via x="17.1704" y="39.0144" extent="1-16" drill="0.6" shape="square"/>
-<wire x1="17.1704" y1="39.0144" x2="17.145" y2="37.1602" width="0.254" layer="16"/>
+<wire x1="16.097" y1="40.1132" x2="17.1704" y2="39.1414" width="0.254" layer="1"/>
+<via x="17.1704" y="39.1414" extent="1-16" drill="0.6" shape="square"/>
+<wire x1="17.1704" y1="39.1414" x2="17.145" y2="37.1602" width="0.254" layer="16"/>
 <wire x1="17.145" y1="37.1602" x2="17.1704" y2="37.1348" width="0.254" layer="16"/>
 </signal>
@@
 <contactref element="PAD1" pad="1"/>
 <wire x1="14.797" y1="43.006" x2="14.797" y2="41.2384" width="0.254" layer="1"/>
-<wire x1="14.797" y1="41.2384" x2="12.573" y2="39.0144" width="0.254" layer="1"/>
-<via x="12.573" y="39.0144" extent="1-16" drill="0.6" shape="square"/>
-<wire x1="12.573" y1="39.0144" x2="12.573" y2="37.1602" width="0.254" layer="16"/>
+<wire x1="14.797" y1="41.2384" x2="12.5476" y2="39.1668" width="0.254" layer="1"/>
+<via x="12.5476" y="39.1668" extent="1-16" drill="0.6" shape="square"/>
+<wire x1="12.5476" y1="39.1668" x2="12.573" y2="37.1602" width="0.254" layer="16"/>
 <wire x1="12.573" y1="37.1602" x2="12.5984" y2="37.1348" width="0.254" layer="16"/>
 </signal>
@@
 <wire x1="24.4475" y1="68.2625" x2="24.209375" y2="68.024375" width="0.8" layer="1"/>
 <wire x1="44.7675" y1="80.9625" x2="44.7675" y2="81.28" width="0.8" layer="1"/>
-<wire x1="42.418" y1="78.5622" x2="42.4053" y2="78.6003" width="0.8" layer="1"/>
-<wire x1="42.4053" y1="78.6003" x2="44.7675" y2="80.9625" width="0.8" layer="1"/>
+<wire x1="41.1734" y1="77.597" x2="44.9707" y2="81.3181" width="0.8" layer="1"/>
+<wire x1="44.9707" y1="81.3181" x2="44.7675" y2="80.9625" width="0.8" layer="1"/>
 <wire x1="44.7675" y1="81.28" x2="44.91" y2="81.28" width="0.8" layer="1"/>
-<wire x1="42.418" y1="78.5622" x2="41.26" y2="77.47" width="0.8" layer="1"/>
+<wire x1="41.1734" y1="77.597" x2="41.26" y2="77.47" width="0.8" layer="1"/>
 <wire x1="43.815" y1="60.96" x2="44.91" y2="60.96" width="0.8" layer="1"/>
 <wire x1="41.275" y1="58.42" x2="43.815" y2="60.96" width="0.8" layer="1"/>
@@
 <wire x1="41.48455" y1="76.8731" x2="41.26" y2="77.47" width="0.8" layer="1"/>
 <wire x1="41.43375" y1="59.055" x2="41.26" y2="58.42" width="0.8" layer="1"/>
-<wire x1="26.19375" y1="77.47" x2="26.19375" y2="82.37855" width="0.8128" layer="1"/>
-<wire x1="26.19375" y1="82.37855" x2="26.924" y2="83.1088" width="0.8128" layer="1"/>
-<wire x1="26.924" y1="83.1088" x2="37.7698" y2="83.1088" width="0.8128" layer="1"/>
-<wire x1="37.7698" y1="83.1088" x2="39.4716" y2="81.407" width="0.8128" layer="1"/>
-<wire x1="39.4716" y1="81.407" x2="42.4053" y2="78.6003" width="0.8128" layer="1"/>
+<wire x1="26.19375" y1="77.47" x2="26.24455" y2="81.31175" width="0.8128" layer="1"/>
+<wire x1="26.24455" y1="81.31175" x2="27.5082" y2="82.7532" width="0.8128" layer="1"/>
+<wire x1="27.5082" y1="82.7532" x2="36.1442" y2="82.7532" width="0.8128" layer="1"/>
+<wire x1="36.1442" y1="82.7532" x2="37.4396" y2="81.3308" width="0.8128" layer="1"/>
+<wire x1="37.4396" y1="81.3308" x2="44.9707" y2="81.3181" width="0.8128" layer="1"/>
 </signal>
 <signal name="X-STOP">
@@
 <contactref element="PAD3" pad="1"/>
 <wire x1="15.447" y1="43.006" x2="15.447" y2="39.7294" width="0.254" layer="1"/>
-<wire x1="15.447" y1="39.7294" x2="14.8844" y2="39.0398" width="0.254" layer="1"/>
-<via x="14.8844" y="39.0398" extent="1-16" drill="0.6" shape="square"/>
-<wire x1="14.8844" y1="39.0398" x2="14.859" y2="37.1856" width="0.254" layer="16"/>
+<wire x1="15.447" y1="39.7294" x2="14.859" y2="39.1922" width="0.254" layer="1"/>
+<via x="14.859" y="39.1922" extent="1-16" drill="0.6" shape="square"/>
+<wire x1="14.859" y1="39.1922" x2="14.859" y2="37.1856" width="0.254" layer="16"/>
 <wire x1="14.859" y1="37.1856" x2="14.8844" y2="37.1602" width="0.254" layer="16"/>
 </signal>

Commit message: dark clean and add  raster
Parts:
- moved R14 2.93 mm to (16.4, 20.7), turned to 0 degrees
- moved R6 2.61 mm to (18.3, 11.4), turned to 180 degrees
- moved R10 1.45 mm to (16.2, 16.2), turned to 0 degrees
- moved X-S 0.45 mm to (22.2, 41.1)
- moved Y-S 0.44 mm to (25.1, 41.0)
- moved Z-S 0.41 mm to (27.9, 41.0)
Routing:
- net N$27: track 114.4 -> 83.6 mm, vias 3 -> 4
- net SCL: track 34.4 -> 48.0 mm, vias 2 -> 1
- net 3V3: track 186.3 -> 176.3 mm
- net GND: track 310.4 -> 320.1 mm
- net N$23: track 76.2 -> 81.5 mm, vias 4 -> 1
- net 5V: track 103.8 -> 99.1 mm, vias 2 -> 0
- net E-DIR: track 39.0 -> 42.4 mm, vias 3 -> 1
- net Z-DIR: track 27.4 -> 24.7 mm, vias 1 -> 0
- net SDA: track 27.0 -> 28.7 mm
- net Z-STOP: track 9.91 -> 11.2 mm
- net N$S4: track 89.5 -> 90.7 mm, vias 2 -> 1
- net ENABLE: track 81.1 -> 80.1 mm
- net X-STOP: track 6.42 -> 5.85 mm
- net S-A1: track 21.8 -> 22.3 mm
- net HE0: track 28.1 -> 28.6 mm
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- added copper zone on layer 1, net GND
- added copper zone on layer 16, net GND
- added copper zone on layer 1, net GND1
- added copper zone on layer 16, net GND1
Other:
- outline, holes or cut-outs redrawn
- board text added: "PAD1"
- board text added: "PAD2"
- board text added: "PAD3"
- board text removed: "12V-IN"
- board text removed: "12V-IN2"
- board text removed: "ANALOG"
- board text removed: "AUX1"
- board text removed: "AUX2"
- board text removed: "C1"
- board text removed: "C2"
- board text removed: "C3"
- board text removed: "C4"
- board text removed: "C5"
- board text removed: "C6"
- board text removed: "C8"
- board text removed: "D1"
- board text removed: "EXTRA"
- board text removed: "FAN"
- board text removed: "HB"
- board text removed: "HE"
- board text removed: "IC1"
- board text removed: "JP1"
- board text removed: "JP2"
- board text removed: "JP4"
- board text removed: "JP8"
- board text removed: "LED1"
- board text removed: "LED2"
- board text removed: "LED3"
- board text removed: "LM1117-5V"
- board text removed: "Q1"
- board text removed: "Q2"
- board text removed: "Q3"
- board text removed: "R1"
- board text removed: "R10"
- board text removed: "R11"
- board text removed: "R12"
- board text removed: "R13"
- board text removed: "R14"
- board text removed: "R15"
- board text removed: "R2"
- board text removed: "R3"
- board text removed: "R4"
- board text removed: "R5"
- board text removed: "R6"
- board text removed: "SJ10"
- board text removed: "SJ11"
- board text removed: "SJ12"
- board text removed: "SJ13"
- board text removed: "SJ2"
- board text removed: "SJ3"
- board text removed: "SJ4"
- board text removed: "SJ5"
- board text removed: "SJ6"
- board text removed: "SJ7"
- board text removed: "SJ8"
- board text removed: "SJ9"
- board text removed: "X-MOT"
- board text removed: "X-S"
- board text removed: "Y-S"
- board text removed: "Z-MOT1"
- board text removed: "Z-S"
