File: board/E4m.brd (EAGLE design)
At the start: 49.4 x 100.1 mm, 76 parts, among them IC1 MCP23017SS, Q1 IRL540, Q2 IRL540, Q3 IRL540

Commit message: clean clean clean
Parts:
- moved PAD4 0.33 mm to (13.2, 47.3)
- moved PAD5 0.28 mm to (15.7, 47.2)
Routing:
- net SCL: track 48.0 -> 49.5 mm
Changed lines of the file:
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@@
 <element name="PAD2" library="wirepad" package="SMD1,27-2,54" value="WIREPADSMD1,27-254" x="17.1704" y="37.1348" rot="MR0"/>
 <element name="PAD3" library="wirepad" package="SMD1,27-2,54" value="WIREPADSMD1,27-254" x="14.8844" y="37.1602" rot="MR0"/>
-<element name="PAD4" library="wirepad" package="SMD1,27-2,54" value="WIREPADSMD1,27-254" x="12.8524" y="47.1678"/>
-<element name="PAD5" library="wirepad" package="SMD1,27-2,54" value="WIREPADSMD1,27-254" x="15.4432" y="47.244"/>
+<element name="PAD4" library="wirepad" package="SMD1,27-2,54" value="WIREPADSMD1,27-254" x="13.1699" y="47.251621875"/>
+<element name="PAD5" library="wirepad" package="SMD1,27-2,54" value="WIREPADSMD1,27-254" x="15.720059375" y="47.223678125"/>
 <element name="PAD6" library="wirepad" package="SMD1,27-2,54" value="WIREPADSMD1,27-254" x="17.9832" y="47.2694" rot="R180"/>
 <element name="JP3" library="adafruit" package="1X01-CLEANBIG" value="" x="24.0284" y="85.8266"/>
@@
 <wire x1="16.7386" y1="43.9674" x2="15.621" y2="45.085" width="0.254" layer="1"/>
 <wire x1="15.621" y1="45.085" x2="14.9352" y2="45.085" width="0.254" layer="1"/>
-<wire x1="14.9352" y1="45.085" x2="12.8524" y2="47.1678" width="0.254" layer="1"/>
+<wire x1="14.9352" y1="45.085" x2="13.1699" y2="47.251621875" width="0.254" layer="1"/>
 </signal>
 <signal name="N$26" class="3">
 <contactref element="IC1" pad="4"/>
 <contactref element="PAD5" pad="1"/>
-<wire x1="15.4432" y1="47.244" x2="17.397" y2="45.2902" width="0.254" layer="1"/>
+<wire x1="15.720059375" y1="47.223678125" x2="17.397" y2="45.2902" width="0.254" layer="1"/>
 <wire x1="17.397" y1="45.2902" x2="17.397" y2="43.006" width="0.254" layer="1"/>
 </signal>
@@
 <wire x1="12.1158" y1="45.4914" x2="12.1158" y2="43.0911" width="0.254" layer="1"/>
 <wire x1="11.8872" y1="45.72" x2="12.1158" y2="45.4914" width="0.254" layer="1"/>
-<wire x1="11.8872" y1="48.5775" x2="11.8872" y2="45.72" width="0.254" layer="1"/>
-<wire x1="12.2301" y1="48.9204" x2="11.8872" y2="48.5775" width="0.254" layer="1"/>
-<wire x1="18.7452" y1="48.9204" x2="12.2301" y2="48.9204" width="0.254" layer="1"/>
-<wire x1="20.574" y1="47.0916" x2="18.7452" y2="48.9204" width="0.254" layer="1"/>
+<wire x1="11.93038125" y1="48.4733625" x2="11.8872" y2="45.72" width="0.254" layer="1"/>
+<wire x1="12.7381" y1="49.2379" x2="11.93038125" y2="48.4733625" width="0.254" layer="1"/>
+<wire x1="18.9357" y1="49.25821875" x2="12.7381" y2="49.2379" width="0.254" layer="1"/>
+<wire x1="20.574" y1="47.0916" x2="18.9357" y2="49.25821875" width="0.254" layer="1"/>
 <wire x1="20.574" y1="43.6626" x2="20.574" y2="47.0916" width="0.254" layer="1"/>
-<wire x1="21.717" y1="44.8056" x2="20.574" y2="43.6626" width="0.254" layer="16"/>
-<wire x1="25.4889" y1="44.8056" x2="21.717" y2="44.8056" width="0.254" layer="16"/>
-<wire x1="26.6319" y1="43.6626" x2="25.4889" y2="44.8056" width="0.254" layer="16"/>
+<wire x1="21.541740625" y1="44.876721875" x2="20.574" y2="43.6626" width="0.254" layer="16"/>
+<wire x1="26.23058125" y1="44.87671875" x2="21.541740625" y2="44.876721875" width="0.254" layer="16"/>
+<wire x1="26.6319" y1="43.6626" x2="26.23058125" y2="44.87671875" width="0.254" layer="16"/>
 <wire x1="26.6319" y1="28.1178" x2="26.6319" y2="43.6626" width="0.254" layer="16"/>
-<wire x1="27.2034" y1="27.5463" x2="26.6319" y2="28.1178" width="0.254" layer="16"/>
-<wire x1="27.2034" y1="23.0886" x2="27.2034" y2="27.5463" width="0.254" layer="16"/>
-<wire x1="26.289" y1="22.1742" x2="27.2034" y2="23.0886" width="0.254" layer="16"/>
+<wire x1="27.632659375" y1="27.5463" x2="26.6319" y2="28.1178" width="0.254" layer="16"/>
+<wire x1="27.632659375" y1="23.0886" x2="27.632659375" y2="27.5463" width="0.254" layer="16"/>
+<wire x1="26.289" y1="22.1742" x2="27.632659375" y2="23.0886" width="0.254" layer="16"/>
 <wire x1="12.1158" y1="43.0911" x2="12.197" y2="43.006" width="0.254" layer="1"/>
 <wire x1="26.289" y1="22.1742" x2="26.2" y2="22.06" width="0.254" layer="16"/>
@@
 <wire x1="38.2905" y1="50.7492" x2="38.2906" y2="50.9166" width="0.254" layer="1"/>
 <wire x1="14.1732" y1="44.577" x2="14.1732" y2="43.0911" width="0.254" layer="1"/>
-<wire x1="20.8026" y1="44.577" x2="14.1732" y2="44.577" width="0.254" layer="16"/>
-<wire x1="21.4884" y1="45.2628" x2="20.8026" y2="44.577" width="0.254" layer="16"/>
-<wire x1="30.2895" y1="45.2628" x2="21.4884" y2="45.2628" width="0.254" layer="16"/>
+<wire x1="20.449540625" y1="44.59478125" x2="14.1732" y2="44.577" width="0.254" layer="16"/>
+<wire x1="21.27758125" y1="45.298359375" x2="20.449540625" y2="44.59478125" width="0.254" layer="16"/>
+<wire x1="30.2895" y1="45.2628" x2="21.27758125" y2="45.298359375" width="0.254" layer="16"/>
 <wire x1="31.8897" y1="46.863" x2="30.2895" y2="45.2628" width="0.254" layer="16"/>
 <wire x1="43.6626" y1="46.863" x2="38.2905" y2="46.863" width="0.254" layer="16"/>

Commit message: update more and more :(
agrrr
Connections:
- net 3V3: now also IC1.18
- net Z-STEP1: now also JP8.2
Routing:
- net Z-STEP1: track 0.00 -> 22.3 mm, vias 0 -> 3
- net 3V3: track 176.3 -> 189.9 mm, vias 4 -> 5
- net Z-STOP: track 11.2 -> 9.85 mm
- net Y-STOP: track 8.65 -> 8.06 mm
Changed lines of the file:
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@@
 <wire x1="18.75" y1="36.625" x2="18.75" y2="35.875" width="0.254" layer="1"/>
 <wire x1="19.375" y1="37.25" x2="18.75" y2="36.625" width="0.254" layer="1"/>
-<wire x1="25" y1="37.25" x2="19.375" y2="37.25" width="0.254" layer="1"/>
-<wire x1="25" y1="38.375" x2="25" y2="37.25" width="0.254" layer="1"/>
+<wire x1="24.0119375" y1="37.214440625" x2="19.375" y2="37.25" width="0.254" layer="1"/>
+<wire x1="25" y1="38.375" x2="24.0119375" y2="37.214440625" width="0.254" layer="1"/>
 <wire x1="18.75" y1="35.875" x2="18.697" y2="35.756" width="0.254" layer="1"/>
 <wire x1="25" y1="38.375" x2="25.0954" y2="38.4654" width="0.254" layer="1"/>
@@
 <contactref element="Z-S" pad="1"/>
 <contactref element="IC1" pad="28"/>
-<wire x1="27.875" y1="35.875" x2="19.375" y2="35.875" width="0.254" layer="1"/>
-<wire x1="27.875" y1="38.375" x2="27.875" y2="35.875" width="0.254" layer="1"/>
+<wire x1="25.754103125" y1="35.875" x2="19.375" y2="35.875" width="0.254" layer="1"/>
+<wire x1="27.875" y1="38.375" x2="25.754103125" y2="35.875" width="0.254" layer="1"/>
 <wire x1="19.375" y1="35.875" x2="19.347" y2="35.756" width="0.254" layer="1"/>
 <wire x1="27.875" y1="38.375" x2="27.9068" y2="38.4384" width="0.254" layer="1"/>
@@
 <wire x1="12.7381" y1="49.2379" x2="11.93038125" y2="48.4733625" width="0.254" layer="1"/>
 <wire x1="18.9357" y1="49.25821875" x2="12.7381" y2="49.2379" width="0.254" layer="1"/>
-<wire x1="20.574" y1="47.0916" x2="18.9357" y2="49.25821875" width="0.254" layer="1"/>
-<wire x1="20.574" y1="43.6626" x2="20.574" y2="47.0916" width="0.254" layer="1"/>
-<wire x1="21.541740625" y1="44.876721875" x2="20.574" y2="43.6626" width="0.254" layer="16"/>
+<wire x1="20.469859375" y1="47.124621875" x2="18.9357" y2="49.25821875" width="0.254" layer="1"/>
+<wire x1="20.4698625" y1="43.62958125" x2="20.469859375" y2="47.124621875" width="0.254" layer="1"/>
+<wire x1="21.541740625" y1="44.876721875" x2="20.4698625" y2="43.62958125" width="0.254" layer="16"/>
 <wire x1="26.23058125" y1="44.87671875" x2="21.541740625" y2="44.876721875" width="0.254" layer="16"/>
 <wire x1="26.6319" y1="43.6626" x2="26.23058125" y2="44.87671875" width="0.254" layer="16"/>
@@
 <wire x1="12.1158" y1="43.0911" x2="12.197" y2="43.006" width="0.254" layer="1"/>
 <wire x1="26.289" y1="22.1742" x2="26.2" y2="22.06" width="0.254" layer="16"/>
-<via x="20.574" y="43.6626" extent="1-16" drill="0.6096"/>
+<via x="20.4698625" y="43.62958125" extent="1-16" drill="0.6096"/>
 </signal>
 <signal name="HE0">
@@
 <contactref element="ANALOG" pad="3"/>
 <contactref element="IC1" pad="1"/>
-<wire x1="19.3675" y1="45.4025" x2="19.3675" y2="43.02125" width="0.254" layer="1"/>
-<wire x1="19.685" y1="45.72" x2="19.3675" y2="45.4025" width="0.254" layer="1"/>
-<wire x1="21.9075" y1="45.72" x2="19.685" y2="45.72" width="0.254" layer="16"/>
+<wire x1="19.3675" y1="45.702221875" x2="19.3675" y2="43.02125" width="0.254" layer="1"/>
+<wire x1="21.9075" y1="45.72" x2="19.3675" y2="45.702221875" width="0.254" layer="16"/>
 <wire x1="27.78125" y1="51.59375" x2="21.9075" y2="45.72" width="0.254" layer="16"/>
 <wire x1="27.78125" y1="53.6575" x2="27.78125" y2="51.59375" width="0.254" layer="16"/>
@@
 <wire x1="19.3675" y1="43.02125" x2="19.347" y2="43.006" width="0.254" layer="1"/>
 <wire x1="26.82875" y1="54.61" x2="26.6768" y2="54.6564" width="0.254" layer="16"/>
-<via x="19.685" y="45.72" extent="1-16" drill="0.6096"/>
+<via x="19.3675" y="45.702221875" extent="1-16" drill="0.6096"/>
 </signal>
 <signal name="AUX2" class="3">
@@
 <wire x1="38.2905" y1="50.7492" x2="38.2906" y2="50.9166" width="0.254" layer="1"/>
 <wire x1="14.1732" y1="44.577" x2="14.1732" y2="43.0911" width="0.254" layer="1"/>
-<wire x1="20.449540625" y1="44.59478125" x2="14.1732" y2="44.577" width="0.254" layer="16"/>
+<wire x1="20.449540625" y1="44.59478125" x2="15.87476875" y2="44.581821875" width="0.254" layer="16"/>
+<wire x1="15.87476875" y1="44.581821875" x2="14.1732" y2="44.577" width="0.254" layer="16"/>
 <wire x1="21.27758125" y1="45.298359375" x2="20.449540625" y2="44.59478125" width="0.254" layer="16"/>
 <wire x1="30.2895" y1="45.2628" x2="21.27758125" y2="45.298359375" width="0.254" layer="16"/>
@@
 <via x="38.2905" y="46.7487" extent="1-16" drill="0.6096"/>
 <via x="38.9763" y="66.294" extent="1-16" drill="0.6096"/>
+<contactref element="IC1" pad="18"/>
+<wire x1="12.875" y1="34.875" x2="12.875" y2="35.75" width="0.254" layer="1"/>
+<wire x1="13.5" y1="34.25" x2="12.875" y2="34.875" width="0.254" layer="1"/>
+<wire x1="14.375" y1="34.25" x2="13.5" y2="34.25" width="0.254" layer="16"/>
+<wire x1="15.875" y1="35.75" x2="14.375" y2="34.25" width="0.254" layer="16"/>
+<wire x1="15.875" y1="44.5" x2="15.875" y2="35.75" width="0.254" layer="16"/>
+<wire x1="12.875" y1="35.75" x2="12.847" y2="35.756" width="0.254" layer="1"/>
+<wire x1="15.875" y1="44.5" x2="15.87476875" y2="44.581821875" width="0.254" layer="16"/>
+<via x="13.5" y="34.25" extent="1-16" drill="0.6096"/>
 </signal>
 <signal name="HB0">
@@
 <contactref element="U$6" pad="2A"/>
 <wire x1="12.54125" y1="98.7425" x2="11.7475" y2="98.7425" width="0.4" layer="1"/>
-<wire x1="17.62125" y1="93.6625" x2="12.54125" y2="98.7425" width="0.4" layer="1"/>
-<wire x1="23.01875" y1="93.6625" x2="17.62125" y2="93.6625" width="0.4" layer="1"/>
-<wire x1="27.94" y1="88.74125" x2="23.01875" y2="93.6625" width="0.4" layer="1"/>
+<wire x1="17.51203125" y1="93.807278125" x2="12.54125" y2="98.7425" width="0.4" layer="1"/>
+<wire x1="22.90953125" y1="93.807278125" x2="17.51203125" y2="93.807278125" width="0.4" layer="1"/>
+<wire x1="27.94" y1="88.74125" x2="22.90953125" y2="93.807278125" width="0.4" layer="1"/>
 <wire x1="11.7475" y1="98.7425" x2="11.605" y2="98.743" width="0.4" layer="1"/>
 <wire x1="27.94" y1="88.74125" x2="28.0508" y2="88.6226" width="0.4" layer="1"/>
@@
 <contactref element="Z-MOT1" pad="3"/>
 <contactref element="U$6" pad="1A"/>
-<wire x1="15.08125" y1="98.7425" x2="14.2875" y2="98.7425" width="0.4" layer="1"/>
-<wire x1="19.05" y1="94.77375" x2="15.08125" y2="98.7425" width="0.4" layer="1"/>
-<wire x1="24.4475" y1="94.77375" x2="19.05" y2="94.77375" width="0.4" layer="1"/>
-<wire x1="27.94" y1="91.28125" x2="24.4475" y2="94.77375" width="0.4" layer="1"/>
+<wire x1="14.461490625" y1="98.376740625" x2="14.2875" y2="98.7425" width="0.4" layer="1"/>
+<wire x1="18.02384375" y1="94.700090625" x2="14.461490625" y2="98.376740625" width="0.4" layer="1"/>
+<wire x1="24.411940625" y1="94.664528125" x2="18.02384375" y2="94.700090625" width="0.4" layer="1"/>
+<wire x1="27.94" y1="91.28125" x2="24.411940625" y2="94.664528125" width="0.4" layer="1"/>
 <wire x1="14.2875" y1="98.7425" x2="14.145" y2="98.743" width="0.4" layer="1"/>
 <wire x1="27.94" y1="91.28125" x2="28.0508" y2="91.1626" width="0.4" layer="1"/>
@@
 <contactref element="Z-MOT1" pad="4"/>
 <contactref element="U$6" pad="1B"/>
-<wire x1="17.62125" y1="98.7425" x2="16.8275" y2="98.7425" width="0.4" layer="1"/>
-<wire x1="20.955" y1="95.40875" x2="17.62125" y2="98.7425" width="0.4" layer="1"/>
-<wire x1="26.3525" y1="95.40875" x2="20.955" y2="95.40875" width="0.4" layer="1"/>
+<wire x1="16.889728125" y1="98.633278125" x2="16.8275" y2="98.7425" width="0.4" layer="1"/>
+<wire x1="19.5300625" y1="95.40875" x2="16.889728125" y2="98.633278125" width="0.4" layer="1"/>
+<wire x1="26.3525" y1="95.40875" x2="19.5300625" y2="95.40875" width="0.4" layer="1"/>
 <wire x1="27.94" y1="93.82125" x2="26.3525" y2="95.40875" width="0.4" layer="1"/>
 <wire x1="16.8275" y1="98.7425" x2="16.685" y2="98.743" width="0.4" layer="1"/>
@@
 <signal name="Z-STEP1">
 <contactref element="U$6" pad="STEP"/>
+<contactref element="JP8" pad="2"/>
+<wire x1="19.125" y1="86.75" x2="19.125" y2="86.125" width="0.254" layer="1"/>
+<wire x1="16.875" y1="89" x2="19.125" y2="86.75" width="0.254" layer="1"/>
+<wire x1="12.5" y1="93.375" x2="16.875" y2="89" width="0.254" layer="16"/>
+<wire x1="9.5" y1="93.375" x2="12.5" y2="93.375" width="0.254" layer="16"/>
+<wire x1="9" y1="92.875" x2="9.5" y2="93.375" width="0.254" layer="16"/>
+<wire x1="8.6148375" y1="93.17888125" x2="9" y2="92.875" width="0.254" layer="1"/>
+<wire x1="7" y1="93.2017375" x2="8.6148375" y2="93.17888125" width="0.254" layer="1"/>
+<wire x1="5.170021875" y1="93.201740625" x2="7" y2="93.2017375" width="0.254" layer="16"/>
+<wire x1="1.625" y1="96" x2="5.170021875" y2="93.201740625" width="0.254" layer="16"/>
+<wire x1="19.125" y1="86.125" x2="19.225" y2="86.043" width="0.254" layer="1"/>
+<wire x1="1.625" y1="96" x2="1.6" y2="96.01" width="0.254" layer="16"/>
+<via x="16.875" y="89" extent="1-16" drill="0.6096"/>
+<via x="9" y="92.875" extent="1-16" drill="0.6096"/>
+<via x="7" y="93.2017375" extent="1-16" drill="0.6096"/>
 </signal>
 <signal name="N$49">

Commit message: again
Routing:
- net GND: track 320.1 -> 323.0 mm
Changed lines of the file:
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@@
 <wire x1="36.195" y1="58.42" x2="35.86" y2="58.42" width="0.254" layer="1"/>
 <wire x1="38.735" y1="75.565" x2="38.768646875" y2="75.61784375" width="0.254" layer="1"/>
-<wire x1="13.875" y1="60.375" x2="13.125" y2="61.125" width="0.254" layer="1"/>
-<wire x1="13.875" y1="60.25" x2="13.875" y2="60.375" width="0.254" layer="1"/>
-<wire x1="14.125" y1="60" x2="13.875" y2="60.25" width="0.254" layer="1"/>
-<wire x1="18.5" y1="60" x2="14.859" y2="60" width="0.254" layer="1"/>
-<wire x1="14.859" y1="60" x2="14.125" y2="60" width="0.254" layer="1"/>
-<wire x1="18.5" y1="61.125" x2="18.5" y2="60" width="0.254" layer="1"/>
+<wire x1="13.113" y1="60.5274" x2="13.125" y2="61.125" width="0.254" layer="1"/>
+<wire x1="13.14348125" y1="59.642940625" x2="13.113" y2="60.5274" width="0.254" layer="1"/>
+<wire x1="14.91748125" y1="59.6672625" x2="13.14348125" y2="59.642940625" width="0.254" layer="1"/>
+<wire x1="18.46951875" y1="59.667259375" x2="16.807178125" y2="59.697740625" width="0.254" layer="1"/>
+<wire x1="16.807178125" y1="59.697740625" x2="14.91748125" y2="59.6672625" width="0.254" layer="1"/>
+<wire x1="18.5" y1="61.125" x2="18.46951875" y2="59.667259375" width="0.254" layer="1"/>
 <wire x1="13.125" y1="61.125" x2="13.07" y2="61.13" width="0.254" layer="1"/>
 <wire x1="18.5" y1="61.125" x2="18.55" y2="61.13" width="0.254" layer="1"/>
@@
 <wire x1="27.3177" y1="70.7517" x2="27.36" y2="70.76" width="0.254" layer="16"/>
 <wire x1="21.2598" y1="70.5231" x2="21.16" y2="70.56" width="0.254" layer="16"/>
-<wire x1="14.859" y1="59.6646" x2="14.859" y2="60" width="0.254" layer="1"/>
+<wire x1="14.859" y1="59.6646" x2="16.807178125" y2="59.697740625" width="0.254" layer="1"/>
 <wire x1="14.859" y1="59.6646" x2="14.75" y2="59.6646" width="0.254" layer="16"/>
 <wire x1="17.3736" y1="27.6606" x2="17.3736" y2="20.8026" width="0.254" layer="1"/>
@@
 <contactref element="U$3" pad="STEP"/>
 <contactref element="U$5" pad="D3"/>
-<wire x1="26.3525" y1="18.25625" x2="26.3525" y2="16.98625" width="0.254" layer="1"/>
-<wire x1="31.115" y1="23.01875" x2="26.3525" y2="18.25625" width="0.254" layer="1"/>
-<wire x1="31.115" y1="24.4475" x2="31.115" y2="23.01875" width="0.254" layer="1"/>
-<wire x1="32.0675" y1="25.4" x2="31.115" y2="24.4475" width="0.254" layer="1"/>
+<wire x1="29.96438125" y1="20.00123125" x2="26.3525" y2="16.98625" width="0.254" layer="1"/>
+<wire x1="29.9212" y1="22.068790625" x2="29.96438125" y2="20.00123125" width="0.254" layer="1"/>
+<wire x1="29.936440625" y1="23.55088125" x2="29.9212" y2="22.068790625" width="0.254" layer="1"/>
+<wire x1="32.0675" y1="25.4" x2="29.936440625" y2="23.55088125" width="0.254" layer="1"/>
 <wire x1="26.3525" y1="16.98625" x2="26.2" y2="16.98" width="0.254" layer="1"/>
 <wire x1="32.0675" y1="25.4" x2="32.21" y2="25.4" width="0.254" layer="1"/>
@@
 <contactref element="U$5" pad="D2"/>
 <wire x1="26.25" y1="20.625" x2="26.25" y2="19.625" width="0.254" layer="16"/>
-<wire x1="29.125" y1="23.5" x2="26.25" y2="20.625" width="0.254" layer="16"/>
-<wire x1="29.125" y1="39.125" x2="29.125" y2="23.5" width="0.254" layer="16"/>
-<wire x1="28.875" y1="39.375" x2="29.125" y2="39.125" width="0.254" layer="16"/>
-<wire x1="28.875" y1="40.25" x2="28.875" y2="39.375" width="0.254" layer="16"/>
-<wire x1="31.125" y1="42.5" x2="28.875" y2="40.25" width="0.254" layer="16"/>
+<wire x1="29.2012" y1="23.5" x2="26.25" y2="20.625" width="0.254" layer="16"/>
+<wire x1="29.208821875" y1="38.848134375" x2="29.2012" y2="23.5" width="0.254" layer="16"/>
+<wire x1="28.872459375" y1="39.35975625" x2="29.208821875" y2="38.848134375" width="0.254" layer="16"/>
+<wire x1="28.872459375" y1="40.227140625" x2="28.872459375" y2="39.35975625" width="0.254" layer="16"/>
+<wire x1="31.125" y1="42.5" x2="28.872459375" y2="40.227140625" width="0.254" layer="16"/>
 <wire x1="31.125" y1="44.625" x2="31.125" y2="42.5" width="0.254" layer="16"/>
 <wire x1="32.125" y1="45.625" x2="31.125" y2="44.625" width="0.254" layer="16"/>

Commit message: update
Routing:
- net ANALOG: track 49.5 -> 50.1 mm
- net N$55: track 12.7 -> 12.8 mm, vias 0 -> 1
Other:
- board text added: "+"
- board text added: "-"
- board text added: "XS YS ZS"

Commit message: clean
Routing:
- net 3V3: track 189.7 -> 190.4 mm
- net X-DIR: track 40.8 -> 41.4 mm

Commit message: test
Parts:
- moved IC1 0.48 mm to (15.2, 38.9)
- moved SJ15 0.32 mm to (12.5, 91.2)
- moved SJ17 0.18 mm to (15.2, 91.2)
- moved PAD3 0.10 mm to (14.8, 37.1)
Routing:
- net GND: track 323.0 -> 326.2 mm
- net Z-DIR: track 24.7 -> 27.0 mm
- net S-A0: track 17.1 -> 19.2 mm
- net 12V: track 173.1 -> 175.1 mm
- net S-A1: track 22.3 -> 24.2 mm
- net E-DIR: track 42.4 -> 44.1 mm
- net SDA: track 28.7 -> 29.9 mm
- net 3V3: track 190.4 -> 191.3 mm
- net Y-DIR: track 26.1 -> 26.9 mm
- net N$19: track 4.29 -> 4.83 mm
- net 3V31: track 26.0 -> 26.5 mm
- net N$21: track 6.36 -> 5.85 mm
- net N$22: track 6.03 -> 6.53 mm
Other:
- board text added: "12V-IN"
- board text added: "12V-IN1"
- board text added: "ANALOG"
- board text added: "C1"
- board text added: "C2"
- board text added: "C3"
- board text added: "C4"
- board text added: "C5"
- board text added: "C6"
- board text added: "C8"
- board text added: "D1"
- board text added: "D2"
- board text added: "E"
- board text added: "E-MOT"
- board text added: "FAN"
- board text added: "HB"
- board text added: "HE"
- board text added: "HS3 HS1 HS2"
- board text added: "IC1"
- board text added: "JP1"
- board text added: "JP2"
- board text added: "JP3"
- board text added: "JP4"
- board text added: "JP8"
- board text added: "LED1"
- board text added: "LED2"
- board text added: "LED3"
- board text added: "LM1117-5V"
- board text added: "PAD4"
- board text added: "PAD5"
- board text added: "PAD6"
- board text added: "Q1"
- board text added: "Q2"
- board text added: "Q3"
- board text added: "R10"
- board text added: "R12"
- board text added: "R14"
- board text added: "R15"
- board text added: "R4"
- board text added: "R5"
- board text added: "R6"
- board text added: "S"
- board text added: "SJ10"
- board text added: "SJ11"
- board text added: "SJ12"
- board text added: "SJ13"
- board text added: "SJ15"
- board text added: "SJ17"
- board text added: "SJ18"
- board text added: "SJ2"
- board text added: "SJ3"
- board text added: "SJ4"
- board text added: "SJ5"
- board text added: "SJ6"
- board text added: "SJ7"
- board text added: "SJ8"
- board text added: "SJ9"
- board text added: "T0"
- board text added: "T1"
- board text added: "X"
- board text added: "X-MOT"
- board text added: "X-S"
- board text added: "Y"
- board text added: "Y-MOT"
- board text added: "Y-S"
- board text added: "Z"
- board text added: "Z-MOT"
- board text added: "Z-MOT1"
- board text added: "Z-S"
